File: tesis_bku.sch (KiCad schematic (older format))
At the start: 20 parts, among them J1 Connector_RJ10, J10 Connector_Generic_Conn_01x02, J2 Connector_RJ10, J3 Connector_RJ10, J4 Connector_RJ10, J5 Connector_RJ10, J6 Connector_RJ10, J7 Connector_RJ10, J8 Connector_RJ10, J9 Connector_Generic_Conn_01x08, Q1 BC337, Q2 Triac_Thyristor_Mac97a8, U1 ESP32-WROOM, U2 Interface_Expansion_PCF8574, U3 Interface_Expansion_TCA9548AP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, U4 MOC3041M

Commit message: Avance PCB [11/09/21]
    # Agrego avance inputs, outpus.
    # Se corrige referencia de esquematico Power.
Parts:
- removed Q1: BC337, symbol v0-rescue:BC337-00_lib_sch
- added Q?: Transistor_BJT_BC338, symbol 00_lib_sch:Transistor_BJT_BC338
- renumbered C2 to C?, C1 to C?
Other:
- moved on the sheet: U4
Changed lines of the file:
@@
 $Descr A4 11693 8268
 encoding utf-8
-Sheet 1 2
+Sheet 1 1
 Title ""
 Date ""
@@
 $EndComp
 $Comp
-L v0-rescue:BC337-00_lib_sch Q1
-U 1 1 60FC0A3B
-P 4000 3100
-F 0 "Q1" H 4191 3146 50  0000 L CNN
-F 1 "BC337" H 4191 3055 50  0000 L CNN
-F 2 "" H 4200 3025 50  0001 L CIN
-F 3 "" H 4000 3100 50  0001 L CNN
-	1    4000 3100
-	1    0    0    -1
-$EndComp
-$Comp
 L 00_lib_sch:MOC3041M U4
 U 1 1 60FC1318
-P 5300 3300
-F 0 "U4" H 5300 3625 50  0000 C CNN
-F 1 "MOC3041M" H 5300 3534 50  0000 C CNN
-F 2 "" H 5100 3100 50  0001 L CIN
-F 3 "" H 5300 3300 50  0001 L CNN
-	1    5300 3300
+P 5400 3100
+F 0 "U4" H 5400 3425 50  0000 C CNN
+F 1 "MOC3041M" H 5400 3334 50  0000 C CNN
+F 2 "" H 5200 2900 50  0001 L CIN
+F 3 "" H 5400 3100 50  0001 L CNN
+	1    5400 3100
 	1    0    0    -1
 $EndComp
@@
 $EndComp
 $Comp
-L Device:C C2
+L Device:C C?
 U 1 1 6122D0A6
 P 2800 3100
-F 0 "C2" H 2915 3146 50  0000 L CNN
+F 0 "C?" H 2915 3146 50  0000 L CNN
 F 1 "C" H 2915 3055 50  0000 L CNN
 F 2 "" H 2838 2950 50  0001 C CNN
@@
 $EndComp
 $Comp
-L Device:CP C1
+L Device:CP C?
 U 1 1 6122DC39
 P 2450 3100
-F 0 "C1" H 2568 3146 50  0000 L CNN
+F 0 "C?" H 2568 3146 50  0000 L CNN
 F 1 "CP" H 2568 3055 50  0000 L CNN
 F 2 "" H 2488 2950 50  0001 C CNN
@@
 	1    0    0    -1
 $EndComp
-$Sheet
-S 1100 5950 2500 1500
-U 61391A6D
-F0 "Sheet61391A6C" 50
-F1 "Fuente.sch" 50
-$EndSheet
+$Comp
+L 00_lib_sch:Transistor_BJT_BC338 Q?
+U 1 1 612B23BC
+P 3950 3100
+F 0 "Q?" H 4140 3146 50  0000 L CNN
+F 1 "Transistor_BJT_BC338" H 4150 3050 50  0000 L CNN
+F 2 "" H 4150 3025 50  0001 L CIN
+F 3 "" H 3950 3100 50  0001 L CNN
+	1    3950 3100
+	1    0    0    -1
+$EndComp
 $EndSCHEMATC
