File: Fuente.sch (KiCad schematic (older format))
At the start: 11 parts, among them J1 Conn_01x02, J2 Conn_01x02, U1 XL4005E1

Commit message: Avance PCB [11/09/21]
    # Agrego avance inputs, outpus.
    # Se corrige referencia de esquematico Power.
Parts:
- removed D1: 1N5824, symbol 1N5824:1N5824
- removed J1, J2: Conn_01x02, symbol Connector_Generic:Conn_01x02
- removed U1: XL4005E1, symbol xl4005e1:XL4005E1
- added D?: 1N5824, DIOAD1898W129L762D1143, symbol 00_lib_sch:1N5824
- added U?: XL4005E1, symbol 00_lib_sch:XL4005E1
Connections:
- net labels added: [+3V3DC], [+5VDC], [24VAC_in], [AGND], [GND_out]
- net labels removed: Gnd, In, Out
- wire segments 48 -> 38
Other:
- note added: "INVESTIGAR REGULADOR O \nFUENTE SWTH, 3,3V PARA\nSENSORES y ESP32"
Changed lines of the file:
@@
 $Descr A4 11693 8268
 encoding utf-8
-Sheet 2 2
+Sheet 5 5
 Title ""
 Date ""
@@
 $EndComp
 $Comp
-L xl4005e1:XL4005E1 U1
-U 1 1 613951E7
-P 5100 3850
-F 0 "U1" H 5694 4103 60  0000 L CNN
-F 1 "XL4005E1" H 5694 3997 60  0000 L CNN
-F 2 "" H 5100 3850 60  0001 C CNN
-F 3 "" H 5100 3850 60  0000 C CNN
-F 4 "N01-0001" H 5350 3650 50  0000 C BNN "Part"
-	1    5100 3850
-	1    0    0    -1
-$EndComp
-$Comp
-L 1N5824:1N5824 D1
-U 1 1 613925E0
-P 6600 3750
-F 0 "D1" V 6646 3670 50  0000 R CNN
-F 1 "1N5824" V 6555 3670 50  0000 R CNN
-F 2 "" H 6600 3750 50  0000 L BNN
-F 3 "" H 6600 3750 50  0001 L BNN
-F 4 "2" H 6600 3750 50  0001 L BNN "PARTREV"
-F 5 "Microsemi" H 6600 3750 50  0001 L BNN "MANUFACTURER"
-F 6 "IPC 7351B" H 6600 3750 50  0001 L BNN "STANDARD"
-F 7 "13.43mm" H 6600 3750 50  0001 L BNN "MAXIMUM_PACKAGE_HEIGHT"
-	1    6600 3750
-	0    -1   -1   0
-$EndComp
-$Comp
 L Device:CP1 C4
 U 1 1 6139DAFE
@@
 $EndComp
 Wire Wire Line
-	5100 4350 6600 4350
-Wire Wire Line
 	6600 4350 6600 3950
 Connection ~ 5100 4350
@@
 Wire Wire Line
 	4550 3550 4550 3750
-Wire Wire Line
-	5100 4250 5100 4350
-Connection ~ 4550 3550
 $Comp
 L power:GND #PWR01
@@
 Wire Wire Line
 	3600 4100 3600 4350
-Connection ~ 3600 4350
 Wire Wire Line
 	3600 4350 4050 4350
-$Comp
-L Connector_Generic:Conn_01x02 J1
-U 1 1 613D37FA
-P 2850 3900
-F 0 "J1" H 2768 4117 50  0000 C CNN
-F 1 "Conn_01x02" H 2768 4026 50  0000 C CNN
-F 2 "" H 2850 3900 50  0001 C CNN
-F 3 "~" H 2850 3900 50  0001 C CNN
-	1    2850 3900
-	-1   0    0    -1
-$EndComp
-$Comp
-L Connector_Generic:Conn_01x02 J2
-U 1 1 613D5B1C
-P 8100 3700
-F 0 "J2" H 8180 3692 50  0000 L CNN
-F 1 "Conn_01x02" H 8180 3601 50  0000 L CNN
-F 2 "" H 8100 3700 50  0001 C CNN
-F 3 "~" H 8100 3700 50  0001 C CNN
-	1    8100 3700
-	1    0    0    -1
-$EndComp
-Wire Wire Line
-	7250 3200 7900 3200
-Wire Wire Line
-	7900 3200 7900 3700
-Wire Wire Line
-	7900 3800 7900 4350
-Wire Wire Line
-	7900 4350 7250 4350
 Connection ~ 7250 4350
-Wire Wire Line
-	3050 3900 3050 3550
-Wire Wire Line
-	3050 3550 3600 3550
 Connection ~ 3600 3550
-Wire Wire Line
-	3050 4000 3050 4350
-Wire Wire Line
-	3050 4350 3600 4350
 Wire Wire Line
 	5100 3050 5100 2850
@@
 Wire Notes Line
 	2350 4850 2350 1800
-Text Notes 4400 5200 0    79   ~ 16
+Text Notes 4400 5200 0    79   ~ 0
 Modulo Ajustable de fuente de Alimentación\nDC-DC STEP (5-32 V a 0.8-24 V) - 5A
-Wire Wire Line
-	7850 3000 7900 3000
-Wire Wire Line
-	7900 3000 7900 3200
-Connection ~ 7900 3200
-Wire Wire Line
-	3050 3250 3050 3550
-Connection ~ 3050 3550
-Text HLabel 3000 3250 0    50   Input ~ 0
-In
-Wire Wire Line
-	3000 3250 3050 3250
-Text HLabel 7850 3000 0    50   Input ~ 0
-Out
-Wire Wire Line
-	5100 4350 5100 4450
-Text HLabel 4850 4450 0    50   Input ~ 0
-Gnd
-Wire Wire Line
-	4850 4450 5100 4450
-Connection ~ 5100 4450
-Wire Wire Line
-	5100 4450 5100 4500
+Text HLabel 2050 3550 0    50   Input ~ 0
+[24VAC_in]
+Wire Wire Line
+	2950 4350 3600 4350
+Connection ~ 3600 4350
+Wire Wire Line
+	2050 3550 3600 3550
+Wire Wire Line
+	5100 4350 5100 4500
+Text HLabel 8100 3200 2    50   Output ~ 0
+[+5VDC]
+Wire Wire Line
+	7250 3200 8100 3200
+Text HLabel 8150 4350 2    50   Output ~ 0
+[GND_out]
+Wire Wire Line
+	7250 4350 8150 4350
+Text HLabel 8100 5650 2    50   Output ~ 0
+[+3V3DC]
+Text HLabel 8100 6050 2    50   Output ~ 0
+[GND_out]
+Wire Notes Line
+	6500 5450 7750 5450
+Wire Notes Line
+	7750 5450 7750 6300
+Wire Notes Line
+	7750 6300 6500 6300
+Wire Notes Line
+	6500 6300 6500 5450
+Text Notes 6600 5950 0    50   ~ 0
+INVESTIGAR REGULADOR O \nFUENTE SWTH, 3,3V PARA\nSENSORES  y ESP32
+Text HLabel 1950 4350 0    50   Input ~ 0
+[AGND]
+Wire Wire Line
+	5100 4250 5100 4350
+$Comp
+L 00_lib_sch:1N5824 D?
+U 1 1 61A8C44B
+P 6600 3750
+F 0 "D?" V 6646 3670 50  0000 R CNN
+F 1 "1N5824" V 6555 3670 50  0000 R CNN
+F 2 "DIOAD1898W129L762D1143" H 6600 3750 50  0001 L BNN
+F 3 "" H 6600 3750 50  0001 L BNN
+F 4 "2" H 6600 3750 50  0001 L BNN "PARTREV"
+F 5 "Microsemi" H 6600 3750 50  0001 L BNN "MANUFACTURER"
+F 6 "IPC 7351B" H 6600 3750 50  0001 L BNN "STANDARD"
+F 7 "13.43mm" H 6600 3750 50  0001 L BNN "MAXIMUM_PACKAGE_HEIGHT"
+	1    6600 3750
+	0    -1   -1   0
+$EndComp
+Wire Wire Line
+	5100 4350 6600 4350
+$Comp
+L 00_lib_sch:XL4005E1 U?
+U 1 1 61A8D382
+P 5100 3850
+F 0 "U?" H 5200 4450 60  0000 L CNN
+F 1 "XL4005E1" H 5250 3650 60  0000 L CNN
+F 2 "" H 5100 3850 60  0000 C CNN
+F 3 "" H 5100 3850 60  0000 C CNN
+	1    5100 3850
+	1    0    0    -1
+$EndComp
+Connection ~ 4550 3550
 $EndSCHEMATC

Commit message: actualización
Parts:
- C1: value CP1 -> 470uF/50V
- C2: value CP -> 1uF
- C3: value CP -> 33uF
- C4: value CP2 -> 470uF/50V
- L1: value L_Core_Ferrite -> 33uH/5A
- R1: value R_US -> 2K
- R2: value R_US -> 10.5K
- gave numbers to parts that had none: 2
Other:
- note added: "Funcion de Transferencia realimentación\nVOUT=0.8*(1+R2/R1)"
Changed lines of the file:
@@
 U 1 1 61399376
 P 3600 3950
-F 0 "C1" H 3715 3996 50  0000 L CNN
-F 1 "CP1" H 3715 3905 50  0000 L CNN
+F 0 "C1" H 3400 4000 50  0000 L CNN
+F 1 "470uF/50V" H 3500 3900 50  0000 R CNN
 F 2 "" H 3600 3950 50  0001 C CNN
 F 3 "~" H 3600 3950 50  0001 C CNN
@@
 P 7250 3750
 F 0 "C4" H 7365 3796 50  0000 L CNN
-F 1 "CP2" H 7365 3705 50  0000 L CNN
+F 1 "470uF/50V" H 7365 3705 50  0000 L CNN
 F 2 "" H 7250 3750 50  0001 C CNN
 F 3 "~" H 7250 3750 50  0001 C CNN
@@
 U 1 1 613A086D
 P 6150 2300
-F 0 "C3" H 6268 2346 50  0000 L CNN
-F 1 "CP" H 6268 2255 50  0000 L CNN
+F 0 "C3" V 6300 2250 50  0000 L CNN
+F 1 "33uF" V 6400 2250 50  0000 L CNN
 F 2 "" H 6188 2150 50  0001 C CNN
 F 3 "~" H 6150 2300 50  0001 C CNN
@@
 P 6950 3200
 F 0 "L1" V 6769 3200 50  0000 C CNN
-F 1 "L_Core_Ferrite" V 6860 3200 50  0000 C CNN
+F 1 "33uH/5A" V 6860 3200 50  0000 C CNN
 F 2 "" H 6950 3200 50  0001 C CNN
 F 3 "~" H 6950 3200 50  0001 C CNN
@@
 U 1 1 613BC044
 P 5100 2300
-F 0 "R1" V 4895 2300 50  0000 C CNN
-F 1 "R_US" V 4986 2300 50  0000 C CNN
+F 0 "R1" V 5200 2300 50  0000 C CNN
+F 1 "2K" V 5300 2300 50  0000 C CNN
 F 2 "" V 5140 2290 50  0001 C CNN
 F 3 "~" H 5100 2300 50  0001 C CNN
@@
 U 1 1 613B4622
 P 6150 2850
-F 0 "R2" V 5945 2850 50  0000 C CNN
-F 1 "R_US" V 6036 2850 50  0000 C CNN
+F 0 "R2" V 6250 2850 50  0000 C CNN
+F 1 "10.5K" V 6350 2850 50  0000 C CNN
 F 2 "" V 6190 2840 50  0001 C CNN
 F 3 "~" H 6150 2850 50  0001 C CNN
@@
 P 4050 3950
 F 0 "C2" H 4168 3996 50  0000 L CNN
-F 1 "CP" H 4168 3905 50  0000 L CNN
+F 1 "1uF" H 4168 3905 50  0000 L CNN
 F 2 "" H 4088 3800 50  0001 C CNN
 F 3 "~" H 4050 3950 50  0001 C CNN
@@
 Text HLabel 2050 3550 0    50   Input ~ 0
 [24VAC_in]
-Wire Wire Line
-	2950 4350 3600 4350
 Connection ~ 3600 4350
 Wire Wire Line
@@
 	5100 4250 5100 4350
 $Comp
-L 00_lib_sch:1N5824 D?
+L 00_lib_sch:1N5824 D1
 U 1 1 61A8C44B
 P 6600 3750
-F 0 "D?" V 6646 3670 50  0000 R CNN
+F 0 "D1" V 6646 3670 50  0000 R CNN
 F 1 "1N5824" V 6555 3670 50  0000 R CNN
 F 2 "DIOAD1898W129L762D1143" H 6600 3750 50  0001 L BNN
@@
 	5100 4350 6600 4350
 $Comp
-L 00_lib_sch:XL4005E1 U?
+L 00_lib_sch:XL4005E1 U1
 U 1 1 61A8D382
 P 5100 3850
-F 0 "U?" H 5200 4450 60  0000 L CNN
-F 1 "XL4005E1" H 5250 3650 60  0000 L CNN
+F 0 "U1" H 5200 4450 60  0000 L CNN
+F 1 "XL4005E1" H 5400 3850 60  0000 L CNN
 F 2 "" H 5100 3850 60  0000 C CNN
 F 3 "" H 5100 3850 60  0000 C CNN
@@
 $EndComp
 Connection ~ 4550 3550
+Text Notes 5500 2050 0    50   ~ 0
+Funcion de Transferencia realimentación\nVOUT=0.8*(1+R2/R1)
+Wire Wire Line
+	1950 4350 3600 4350
 $EndSCHEMATC
