File: tesis.sch (KiCad schematic (older format))
At the start: 20 parts, among them J1 Connector_RJ10, J10 Connector_Generic_Conn_01x02, J2 Connector_RJ10, J3 Connector_RJ10, J4 Connector_RJ10, J5 Connector_RJ10, J6 Connector_RJ10, J7 Connector_RJ10, J8 Connector_RJ10, J9 Connector_Generic_Conn_01x08, Q2 Triac_Thyristor_Mac97a8, U1 ESP32-WROOM, U2 Interface_Expansion_PCF8574, U3 Interface_Expansion_TCA9548AP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, U4 MOC3041M

Commit message: Avance PCB [11/09/21]
    # Agrego avance inputs, outpus.
    # Se corrige referencia de esquematico Power.
Parts:
- removed C?: C, symbol Device:C
- removed C?: CP, symbol Device:CP
- removed J1, J2, J3, J4, J5, J6, J7, J8: Connector_RJ10, 00_lib_fp:4P4C_narrow, symbol 00_lib_sch:Connector_RJ10
- removed J10: Connector_Generic_Conn_01x02, symbol 00_lib_sch:Connector_Generic_Conn_01x02
- removed J9: Connector_Generic_Conn_01x08, symbol 00_lib_sch:Connector_Generic_Conn_01x08
- removed MOD1: RPi_GPIO, 00_lib_fp:RPi_fp, symbol 00_lib_sch:RPi_GPIO
- removed Q2: Triac_Thyristor_Mac97a8, symbol 00_lib_sch:Triac_Thyristor_Mac97a8
- removed Q?: Transistor_BJT_BC338, symbol 00_lib_sch:Transistor_BJT_BC338
- removed R1: Device_R_US, symbol 00_lib_sch:Device_R_US
- removed U1: ESP32-WROOM, 00_lib_fp:ESP32-WROOM, symbol 00_lib_sch:ESP32-WROOM
- removed U2: Interface_Expansion_PCF8574, 00_lib_fp:SOIC-16W_7.5x10.3mm_P1.27mm, symbol 00_lib_sch:Interface_Expansion_PCF8574
- removed U3: Interface_Expansion_TCA9548APWR, Package_SO:TSSOP-24_4.4x7.8mm_P0.65mm, symbol 00_lib_sch:Interface_Expansion_TCA9548APWR
- removed U4: MOC3041M, symbol 00_lib_sch:MOC3041M
- added J?: Screw_Terminal_01x02, symbol Connector:Screw_Terminal_01x02
Connections:
- net labels added: +3V3, +5V, 24VAC_IN, AGND_IN, GND
- wire segments 0 -> 6
