File: Outputs.sch (KiCad schematic (older format))
At the start: 0 parts

Commit message: Arreglo raiz de proyecto
Parts:
- added C?: 10u, symbol Device:CP1
- added C?: 100n, symbol Device:C
- added C?: C, symbol Device:C
- added J?: Screw_Terminal_01x02, symbol Connector:Screw_Terminal_01x02
- added J?: Screw_Terminal_01x08, symbol Connector:Screw_Terminal_01x08
- added Q?: Mac97a8, symbol 00_lib_sch:Triac_Thyristor_Mac97a8
- added Q?: Q_NMOS_DGS, symbol Device:Q_NMOS_DGS
- added R? (x6): 10k, symbol Device:R
- added R? (x2): 4k7, symbol Device:R
- added R?: 470, symbol Device:R
- added R? (x2): 1k, symbol Device:R
- added R?: R, symbol Device:R
- added U?: MOC3043, symbol 00_lib_sch:MOC3041M
- added U?: PCF8574, 00_lib_fp:SOIC-16W_7.5x10.3mm_P1.27mm, symbol 00_lib_sch:Interface_Expansion_PCF8574
Connections:
- new net: Q?.2 (G), U?.4
- new net: J?.1 (Pin_1), Q?.3 (MT2), R?.1, R?.1
- new net: Q?.3 (S), R?.1, U?.1
- new net: R?.1, U?.2
- new net: R?.2, U?.6
- new net: R?.1, R?.2, U?.1 (A0)
- new net: R?.1, R?.2, U?.2 (A1)
- new net: R?.1, R?.2, U?.3 (A2)
- new net: C?.1, R?.2
- new net +3V3: C?.1, C?.1, R?.1, R?.1, R?.1, R?.1, R?.1, U?.16 (VDD)
- new net +5V: Q?.1 (D)
- new net GND: C?.2, C?.2, R?.2, R?.2, R?.2, R?.2, R?.2, U?.8 (VSS)
- new net P0: Q?.2 (G), U?.4 (P0)
- new net P1: U?.5 (P1)
- new net P2: U?.6 (P2)
- new net P3: U?.7 (P3)
- new net P4: U?.9 (P4)
- new net P5: U?.10 (P5)
- new net P6: U?.11 (P6)
- new net P7: U?.12 (P7)
- new net [24VAC_in]: Q?.1 (MT1)
- new net [AGND]: C?.2, J?.1 (Pin_1), J?.2 (Pin_2)
- new net [SCL_outputs]: R?.2, U?.14 (SCL)
- new net [SDA_outputs]: R?.2, U?.15 (SDA)
- no-connect marks 0 -> 1
Other:
- note added: "0x20"
- note added: "0x21"
- note added: "0x22"
- note added: "0x23"
- note added: "0x24"
- note added: "0x25"
- note added: "0x26"
- note added: "0x27"
- note added: "A0"
- note added: "A1"
- note added: "A2"
- note added: "Address"
- note added: "Capacitores de desacople.\nColocar lo mas cercano posible \na los pines del IC en cuestion."
- note added: "H"
- note added: "L"
- note added: "Si 24VAC es FASE y Si llamamos \nAGND = NEUTRO entonces está bien"
