File: monitor.sch (KiCad schematic (older format))
At the start: 9 parts, among them U1 ACS712-05, U2 LM358

Commit message: Revision
    * Acomodo los datos de F.Fab y B.Fab
    * Genero ibom
    * Exporto PDF e imagenes
Parts:
- R1: value R -> 1k7; Field4 (none) -> 1%
- R2: value R -> 3k3; Field4 (none) -> 1%
Changed lines of the file:
@@
 U 1 1 6186B0FA
 P 7050 2950
-F 0 "R1" H 7120 2996 50  0000 L CNN
-F 1 "R" H 7120 2905 50  0000 L CNN
+F 0 "R1" H 6875 2975 50  0000 L CNN
+F 1 "1k7" V 7050 2875 50  0000 L CNN
 F 2 "00_lib_fp:R_0805_2012Metric_Pad1.20x1.40mm_HandSolder" V 6980 2950 50  0001 C CNN
 F 3 "" H 7050 2950 50  0001 C CNN
+F 4 "1%" H 6925 2900 50  0000 C CNN "Field4"
 	1    7050 2950
 	1    0    0    -1
@@
 U 1 1 6186B359
 P 7050 3350
-F 0 "R2" H 7120 3396 50  0000 L CNN
-F 1 "R" H 7120 3305 50  0000 L CNN
+F 0 "R2" H 6875 3375 50  0000 L CNN
+F 1 "3k3" V 7050 3275 50  0000 L CNN
 F 2 "00_lib_fp:R_0805_2012Metric_Pad1.20x1.40mm_HandSolder" V 6980 3350 50  0001 C CNN
 F 3 "" H 7050 3350 50  0001 C CNN
+F 4 "1%" H 6925 3300 50  0000 C CNN "Field4"
 	1    7050 3350
 	1    0    0    -1
